File: CameraBoard.brd (EAGLE design)
At the start: 44.5 x 53.1 mm, 17 parts

Commit message: Removed JSTs, updated revision
Parts:
- removed CN1, CN2: (no value), adafruit:JST-PH-2-SMT-RA
- added C1_HIGH, C1_LOW, C2_HIGH, C2_LOW: (no value), adafruit:1X01
Connections:
- net CAM_HIGH: now also C1_HIGH.1, C2_HIGH.1; no longer CN1.1, CN2.1
- net CAM_LOW: now also C1_LOW.1, C2_LOW.1; no longer CN1.2, CN2.2
Routing:
- net CAM_LOW: track 59.3 -> 73.8 mm
- net CAM_HIGH: track 60.8 -> 71.8 mm
Other:
- board text added: "FLIGHT READY - 4/16/19"
- board text removed: "FLIGHT READY - 2/27/19"
Changed lines of the file:
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@@
 <?xml version="1.0" encoding="utf-8"?>
 <!DOCTYPE eagle SYSTEM "eagle.dtd">
-<eagle version="9.3.1">
+<eagle version="9.4.1">
 <drawing>
 <settings>
@@
 <wire x1="44.45" y1="0" x2="44.45" y2="53.086" width="0.254" layer="20"/>
 <wire x1="44.45" y1="53.086" x2="0" y2="53.086" width="0.254" layer="20"/>
-<text x="34.544" y="40.894" size="2.1844" layer="22" rot="MR0">CAMERA BOARD</text>
-<text x="40.894" y="36.576" size="2.1844" layer="22" rot="MR0">FLIGHT READY - 2/27/19</text>
+<text x="12.954" y="6.858" size="2.1844" layer="21">CAMERA BOARD</text>
+<text x="5.588" y="9.144" size="2.1844" layer="21">FLIGHT READY - 4/16/19</text>
 </plain>
 <attributes>
@@
 <attribute name="VALUE" x="23.628" y="45.123" size="1.016" layer="27" rot="R180"/>
 </element>
-<element name="CN1" library="adafruit" library_urn="urn:adsk.eagle:library:420" package="JST-PH-2-SMT-RA" package3d_urn="urn:adsk.eagle:package:6240692/1" value="" x="5.334" y="15.494" smashed="yes" rot="R90">
-<attribute name="NAME" x="9.906" y="8.128" size="1.27" layer="25" font="vector" rot="R90"/>
-<attribute name="VALUE" x="12.954" y="12.954" size="1.27" layer="27" font="vector" rot="R90"/>
-</element>
-<element name="CN2" library="adafruit" library_urn="urn:adsk.eagle:library:420" package="JST-PH-2-SMT-RA" package3d_urn="urn:adsk.eagle:package:6240692/1" value="" x="17.526" y="5.08" smashed="yes" rot="R180">
-<attribute name="NAME" x="25.4" y="9.398" size="1.27" layer="25" font="vector" rot="R180"/>
-<attribute name="VALUE" x="20.066" y="12.7" size="1.27" layer="27" font="vector" rot="R180"/>
-</element>
 <element name="H1" library="holes" library_urn="urn:adsk.eagle:library:237" package="2,8-PAD" package3d_urn="urn:adsk.eagle:package:14281/1" value="MOUNT-PAD-ROUND2.8" x="37.846" y="5.08" smashed="yes"/>
 <element name="H2" library="holes" library_urn="urn:adsk.eagle:library:237" package="2,8-PAD" package3d_urn="urn:adsk.eagle:package:14281/1" value="MOUNT-PAD-ROUND2.8" x="5.334" y="5.08" smashed="yes"/>
@@
 <attribute name="NAME" x="13.97" y="37.846" size="1.27" layer="25"/>
 <attribute name="VALUE" x="13.97" y="32.766" size="1.27" layer="27"/>
+</element>
+<element name="C1_HIGH" library="adafruit" library_urn="urn:adsk.eagle:library:420" package="1X01" value="" x="2.032" y="14.986" smashed="yes">
+<attribute name="NAME" x="0.6858" y="16.8148" size="1.27" layer="25" ratio="10"/>
+<attribute name="VALUE" x="0.762" y="11.811" size="1.27" layer="27"/>
+</element>
+<element name="C1_LOW" library="adafruit" library_urn="urn:adsk.eagle:library:420" package="1X01" value="" x="2.032" y="12.192" smashed="yes">
+<attribute name="NAME" x="0.6858" y="14.0208" size="1.27" layer="25" ratio="10"/>
+<attribute name="VALUE" x="0.762" y="9.017" size="1.27" layer="27"/>
+</element>
+<element name="C2_HIGH" library="adafruit" library_urn="urn:adsk.eagle:library:420" package="1X01" value="" x="13.97" y="1.778" smashed="yes" rot="R90">
+<attribute name="NAME" x="12.1412" y="0.4318" size="1.27" layer="25" ratio="10" rot="R90"/>
+<attribute name="VALUE" x="17.145" y="0.508" size="1.27" layer="27" rot="R90"/>
+</element>
+<element name="C2_LOW" library="adafruit" library_urn="urn:adsk.eagle:library:420" package="1X01" value="" x="16.764" y="1.778" smashed="yes">
+<attribute name="NAME" x="15.4178" y="3.6068" size="1.27" layer="25" ratio="10"/>
+<attribute name="VALUE" x="15.494" y="-1.397" size="1.27" layer="27"/>
 </element>
 </elements>
@@
 <contactref element="H6" pad="B2,8"/>
 <wire x1="36.576" y1="11.176" x2="36.576" y2="16.51" width="0.508" layer="1"/>
-<contactref element="CN1" pad="2"/>
-<contactref element="CN2" pad="2"/>
 <wire x1="9.398" y1="22.774" x2="9.398" y2="21.1046" width="0.508" layer="1"/>
 <via x="9.398" y="21.1046" extent="1-16" drill="0.35"/>
@@
 <via x="18.542" y="13.462" extent="1-16" drill="0.35"/>
 <wire x1="18.542" y1="13.462" x2="18.542" y2="8.78" width="0.508" layer="1"/>
-<wire x1="18.542" y1="8.78" x2="18.526" y2="8.78" width="0.508" layer="1"/>
 <wire x1="18.542" y1="13.462" x2="18.542" y2="11.176" width="0.508" layer="1"/>
 <wire x1="18.542" y1="11.176" x2="36.576" y2="11.176" width="0.508" layer="1"/>
 <wire x1="18.542" y1="13.462" x2="13.97" y2="13.462" width="0.508" layer="16"/>
-<wire x1="13.97" y1="13.462" x2="13.97" y2="14.478" width="0.508" layer="16"/>
-<via x="13.97" y="14.478" extent="1-16" drill="0.35"/>
-<wire x1="13.97" y1="14.478" x2="13.97" y2="14.494" width="0.508" layer="1"/>
-<wire x1="13.97" y1="14.494" x2="9.034" y2="14.494" width="0.508" layer="1"/>
+<contactref element="C1_LOW" pad="1"/>
+<contactref element="C2_LOW" pad="1"/>
+<wire x1="18.542" y1="8.78" x2="18.542" y2="3.556" width="0.6096" layer="1"/>
+<wire x1="18.542" y1="3.556" x2="16.764" y2="1.778" width="0.6096" layer="1"/>
+<wire x1="13.97" y1="13.462" x2="6.858" y2="13.462" width="0.6096" layer="16"/>
+<wire x1="6.858" y1="13.462" x2="5.334" y2="11.938" width="0.6096" layer="16"/>
+<via x="5.334" y="11.938" extent="1-16" drill="0.35"/>
+<wire x1="5.334" y1="11.938" x2="2.286" y2="11.938" width="0.6096" layer="1"/>
+<wire x1="2.286" y1="11.938" x2="2.032" y2="12.192" width="0.6096" layer="1"/>
 </signal>
 <signal name="CAM_HIGH">
@@
 <wire x1="6.858" y1="20.32" x2="11.938" y2="20.32" width="0.508" layer="1"/>
 <wire x1="11.938" y1="20.32" x2="11.938" y2="22.774" width="0.508" layer="1"/>
-<contactref element="CN2" pad="1"/>
-<contactref element="CN1" pad="1"/>
 <wire x1="11.938" y1="20.32" x2="16.526" y2="20.32" width="0.508" layer="1"/>
-<wire x1="16.526" y1="20.32" x2="16.526" y2="8.78" width="0.508" layer="1"/>
-<wire x1="11.938" y1="20.32" x2="11.938" y2="16.494" width="0.508" layer="1"/>
-<wire x1="11.938" y1="16.494" x2="9.034" y2="16.494" width="0.508" layer="1"/>
+<wire x1="11.938" y1="20.32" x2="11.938" y2="16.764" width="0.508" layer="1"/>
+<wire x1="11.938" y1="16.764" x2="11.938" y2="16.494" width="0.508" layer="1"/>
 <wire x1="16.526" y1="20.32" x2="16.526" y2="23.114" width="0.508" layer="1"/>
 <wire x1="16.526" y1="23.114" x2="16.51" y2="23.114" width="0.508" layer="1"/>
@@
 <via x="36.576" y="23.114" extent="1-16" drill="0.35"/>
 <wire x1="36.576" y1="23.114" x2="36.576" y2="28.194" width="0.508" layer="1"/>
+<contactref element="C1_HIGH" pad="1"/>
+<contactref element="C2_HIGH" pad="1"/>
+<wire x1="11.938" y1="16.764" x2="10.16" y2="14.986" width="0.508" layer="1"/>
+<wire x1="10.16" y1="14.986" x2="2.032" y2="14.986" width="0.508" layer="1"/>
+<wire x1="10.16" y1="14.986" x2="10.16" y2="5.588" width="0.6096" layer="1"/>
+<wire x1="10.16" y1="5.588" x2="13.97" y2="1.778" width="0.6096" layer="1"/>
 </signal>
 </signals>
